File: hw/bm/bm.sch (KiCad schematic (older format))
At the start: 50 parts, among them P1 PX0707/06S, P2 PX0707/06S, P3 Deans Male, P4 Deans Male, P5 JST-XH, P6 JST-XH, P7 I²C, P8 I²C, U1 MCP3428, U2 MCP3428

Commit message: Update bm
Parts:
- P3, P4: value Deans Male -> XT60 Male
Connections:
- wire segments 166 -> 162
Other:
- note added: "If the bus lines are twisted-pairs, each bus line\nmust be twisted with a V SS return. Alternatively,\nthe SCL line can be twisted with a V SS return,\nand the SDA line twisted with a V DD return. In\nthe latter case, capacitors must be used to\ndecouple the V DD line to the V SS line at both\nends of the twisted pairs.\n\nExcerpt from page 60 of UM10204"
- note added: "Note on I²C wiring"
- moved on the sheet: C1, C10, C11, C12, C2, C3, C4, C5, C6, C7, C8, C9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

Commit message: Some random changes to the bm
Other:
- note added: "Half blue\nFull blue\nFull brown\nHalf brown"
- note added: "SCL"
- note added: "SDA"
Changed lines of the file:
@@
 Wire Wire Line
 	10350 3750 10350 3300
-Text Notes 9450 2550 0    40   ~ 0
+Text Notes 9450 2275 0    40   ~ 0
 If the bus lines are twisted-pairs, each bus line\nmust be twisted with a V SS return. Alternatively,\nthe SCL line can be twisted with a V SS return,\nand the SDA line twisted with a V DD return. In\nthe latter case, capacitors must be used to\ndecouple the V DD line to the V SS line at both\nends of the twisted pairs.\n\nExcerpt from page 60 of UM10204
-Text Notes 9450 1950 0    60   Italic 12
+Text Notes 9450 1675 0    60   Italic 12
 Note on I²C wiring
 Wire Notes Line
-	9400 1950 11000 1950
+	9400 1675 11000 1675
 Wire Notes Line
-	11000 1950 11000 2550
+	11000 1675 11000 2275
 Wire Notes Line
-	11000 2550 9400 2550
+	11000 2275 9400 2275
 Wire Notes Line
-	9400 2550 9400 1850
+	9400 2275 9400 1575
 Wire Notes Line
-	9400 1850 10300 1850
+	9400 1575 10300 1575
 Wire Notes Line
-	10300 1850 10450 1950
+	10300 1575 10450 1675
 Wire Notes Line
-	9500 2550 9500 2950
+	9500 2275 9500 2950
 Wire Notes Line
 	9500 2950 9650 2950
@@
 	9650 2950 9600 3000
 Wire Notes Line
-	10500 2750 10500 2550
+	10500 2275 10500 2750
 Wire Notes Line
 	10500 2750 10450 2700
 Wire Notes Line
 	10500 2750 10550 2700
+Text Notes 10075 2825 1    60   ~ 0
+Half blue\nFull blue\nFull brown\nHalf brown
+Text Notes 10175 3450 1    60   ~ 0
+SCL
+Text Notes 9700 3450 1    60   ~ 0
+SDA
 $EndSCHEMATC
