File: hw/sssw/sssw.kicad_pcb (KiCad board)
At the start: 2 copper layers, 6 parts, among them P1 INPUT, Q1 SUP85

Commit message: Minor changes to sssw
Parts:
- added G3.5_Bullet_Edge: VAL**, sssw:G3.5_Bullet_Edge, F.Cu at (98.5, 56.0)
- added G3.5_Bullet_Edge: VAL**, sssw:G3.5_Bullet_Edge, F.Cu at (133.0, 50.5)
- added P2: ACTIVATE, Pin_Headers:Pin_Header_Angled_1x02, F.Cu at (121.0, 71.0)
- added P3: OUTPUT, sssw:G3.5_Bullet_Edge, F.Cu at (149.0, 79.0)
- P1: footprint Pin_Headers:Pin_Header_Angled_1x02 -> sssw:G3.5_Bullet_Edge
- moved P1 55.6 mm to (113.0, 79.0), turned to 270 degrees
- moved R3 40.4 mm to (128.8, 75.2), turned to 180 degrees
- moved R1 39.4 mm to (120.0, 76.0), turned to 270 degrees
- moved Q1 39.0 mm to (119.8, 82.5), turned to 270 degrees
- moved R2 37.2 mm to (128.8, 71.8), turned to 180 degrees
- moved D1 24.4 mm to (133.2, 75.2)
Connections:
- Q1 pad D: (no net) -> Net-(P3-Pad2)
- R1 pad 1: (no net) -> Net-(P2-Pad2)
Routing:
- net GND: track 0.00 -> 44.7 mm
- net Net-(P3-Pad2): track 0.00 -> 29.4 mm
- net Net-(Q1-PadG): track 0.00 -> 15.7 mm
- net Net-(P1-Pad2): track 0.00 -> 9.53 mm
- net Net-(P2-Pad2): track 0.00 -> 5.29 mm
- net Net-(D1-Pad1): track 0.00 -> 2.15 mm
Other:
- board outline added: 46 x 39.5 mm

Commit message: minor changes to sssw
Parts:
- removed G3.5_Bullet_Edge (x2): VAL**, sssw:G3.5_Bullet_Edge
- P1: footprint sssw:G3.5_Bullet_Edge -> sssw:G3.5_Bullet_Edge_Short; moved to B.Cu
- P3: footprint sssw:G3.5_Bullet_Edge -> sssw:G3.5_Bullet_Edge_Short
- moved P1 7.00 mm to (106.0, 79.0)
- moved P3 2.00 mm to (151.0, 79.0)
Routing:
- net GND: track 44.7 -> 112.5 mm, vias 0 -> 5
- net Net-(P1-Pad2): track 9.53 -> 52.4 mm, vias 0 -> 5
- net Net-(P3-Pad2): track 29.4 -> 41.6 mm
- net Net-(Q1-PadG): track 15.7 -> 12.9 mm
Other:
- board size 46 x 39.5 mm -> 46 x 21 mm
- net class Default: via_dia 0.889 -> 1.2
- rule via_min_drill: 0.508 -> 0.6
- rule via_min_size: 0.889 -> 1.2
