File: hw/sssw/sssw.sch (KiCad schematic (older format))
At the start: 8 parts, among them P1 INPUT, P2 ACTIVATE, P3 OUTPUT, Q1 SUP85

Commit message: Minor modifications to sssw sch
Other:
- moved on the sheet: P1, P3, Q1
Changed lines of the file:
@@
 encoding utf-8
 Sheet 1 1
-Title ""
+Title "Solid State Safety Switch"
 Date ""
 Rev ""
-Comp ""
+Comp "AAUSHIP"
 Comment1 ""
 Comment2 ""
@@
 L MOSFET_N Q1
 U 1 1 52F79D2B
-P 6300 3850
-F 0 "Q1" H 6250 4000 60  0000 R CNN
-F 1 "SUP85" H 6250 3650 60  0000 R CNN
-F 2 "" H 6300 3850 60  0000 C CNN
-F 3 "" H 6300 3850 60  0000 C CNN
-	1    6300 3850
-	1    0    0    -1
+P 6100 3350
+F 0 "Q1" H 6050 3500 60  0000 R CNN
+F 1 "SUP85" H 6050 3150 60  0000 R CNN
+F 2 "" H 6100 3350 60  0000 C CNN
+F 3 "" H 6100 3350 60  0000 C CNN
+	1    6100 3350
+	0    1    -1   0
 $EndComp
 $Comp
 L CONN_2 P1
 U 1 1 52F7A037
-P 4500 3400
-F 0 "P1" V 4450 3400 40  0000 C CNN
-F 1 "INPUT" V 4550 3400 40  0000 C CNN
-F 2 "" H 4500 3400 60  0000 C CNN
-F 3 "" H 4500 3400 60  0000 C CNN
-	1    4500 3400
+P 4500 3150
+F 0 "P1" V 4450 3150 40  0000 C CNN
+F 1 "INPUT" V 4550 3150 40  0000 C CNN
+F 2 "" H 4500 3150 60  0000 C CNN
+F 3 "" H 4500 3150 60  0000 C CNN
+	1    4500 3150
 	-1   0    0    -1
 $EndComp
@@
 L CONN_2 P3
 U 1 1 52F7A049
-P 6850 3400
-F 0 "P3" V 6800 3400 40  0000 C CNN
-F 1 "OUTPUT" V 6900 3400 40  0000 C CNN
-F 2 "" H 6850 3400 60  0000 C CNN
-F 3 "" H 6850 3400 60  0000 C CNN
-	1    6850 3400
+P 6850 3150
+F 0 "P3" V 6800 3150 40  0000 C CNN
+F 1 "OUTPUT" V 6900 3150 40  0000 C CNN
+F 2 "" H 6850 3150 60  0000 C CNN
+F 3 "" H 6850 3150 60  0000 C CNN
+	1    6850 3150
 	1    0    0    -1
 $EndComp
@@
 L GND #PWR1
 U 1 1 52F7A074
-P 4950 3600
-F 0 "#PWR1" H 4950 3600 30  0001 C CNN
-F 1 "GND" H 4950 3530 30  0001 C CNN
-F 2 "" H 4950 3600 60  0000 C CNN
-F 3 "" H 4950 3600 60  0000 C CNN
-	1    4950 3600
+P 4950 3350
+F 0 "#PWR1" H 4950 3350 30  0001 C CNN
+F 1 "GND" H 4950 3280 30  0001 C CNN
+F 2 "" H 4950 3350 60  0000 C CNN
+F 3 "" H 4950 3350 60  0000 C CNN
+	1    4950 3350
 	1    0    0    -1
 $EndComp
-Wire Wire Line
-	4850 3500 4950 3500
-Wire Wire Line
-	4950 3500 4950 3600
 $Comp
 L R R1
@@
 $EndComp
 $Comp
-L GND #PWR5
-U 1 1 52F7A0CC
-P 6400 4150
-F 0 "#PWR5" H 6400 4150 30  0001 C CNN
-F 1 "GND" H 6400 4080 30  0001 C CNN
-F 2 "" H 6400 4150 60  0000 C CNN
-F 3 "" H 6400 4150 60  0000 C CNN
-	1    6400 4150
-	1    0    0    -1
-$EndComp
-Wire Wire Line
-	4850 3300 6500 3300
-Wire Wire Line
-	5400 3850 6100 3850
-Wire Wire Line
-	5500 3900 5500 3850
-Connection ~ 5500 3850
-Wire Wire Line
-	5500 4500 5500 4400
-$Comp
 L CONN_2 P2
 U 1 1 52F7A13E
@@
 	1    0    0    -1
 $EndComp
-Wire Wire Line
-	4950 4050 4950 4150
-Wire Wire Line
-	4950 4050 4850 4050
-Wire Wire Line
-	6500 3500 6400 3500
-Wire Wire Line
-	6400 3500 6400 3650
-Wire Wire Line
-	6400 4050 6400 4150
-Wire Notes Line
-	5850 3700 5850 4350
-Wire Notes Line
-	5850 4350 7050 4350
-Wire Notes Line
-	7050 4350 7050 3150
-Wire Notes Line
-	7050 3150 4300 3150
-Wire Notes Line
-	4300 3150 4300 3700
-Wire Notes Line
-	4300 3700 5850 3700
-Text Notes 5300 3150 0    60   Italic 0
+Text Notes 5300 2900 0    60   Italic 0
 High Power Path
 $Comp
@@
 	-1   0    0    1
 $EndComp
-Wire Wire Line
-	4900 3850 4850 3850
-Wire Wire Line
-	5750 4450 5750 4400
-Wire Wire Line
-	5750 3900 5750 3850
-Connection ~ 5750 3850
-Wire Wire Line
-	5750 4950 5750 4850
 $Comp
 L GND #PWR4
@@
 	1    0    0    -1
 $EndComp
+Wire Wire Line
+	4850 3250 5900 3250
+Wire Wire Line
+	4950 3250 4950 3350
+Wire Wire Line
+	4850 3050 6500 3050
+Wire Wire Line
+	5400 3850 6100 3850
+Wire Wire Line
+	5500 3900 5500 3850
+Connection ~ 5500 3850
+Wire Wire Line
+	5500 4500 5500 4400
+Wire Wire Line
+	4950 4050 4950 4150
+Wire Wire Line
+	4950 4050 4850 4050
+Wire Wire Line
+	6300 3250 6500 3250
+Wire Notes Line
+	7050 2900 4300 2900
+Wire Notes Line
+	4300 2900 4300 3700
+Wire Wire Line
+	4900 3850 4850 3850
+Wire Wire Line
+	5750 4450 5750 4400
+Wire Wire Line
+	5750 3900 5750 3850
+Connection ~ 5750 3850
+Wire Wire Line
+	5750 4950 5750 4850
+Connection ~ 4950 3250
+Wire Notes Line
+	7050 2900 7050 3700
+Wire Notes Line
+	7050 3700 4300 3700
+Wire Wire Line
+	6100 3850 6100 3550
 $EndSCHEMATC

Commit message: Fix sssw sch
Connections:
- net GND: now also P1.1 (P1), P2.1 (P1), P3.1 (P1); no longer P1.2 (PM), P2.2 (PM), Q1.S
- net at R1.1: now also P2.2 (PM); no longer P2.1 (P1)
- new net: P1.2 (PM), Q1.S
Other:
- note added: "Female\nbullets"
- note added: "Male\nbullets"
Changed lines of the file:
@@
 L GND #PWR1
 U 1 1 52F7A074
-P 4950 3350
-F 0 "#PWR1" H 4950 3350 30  0001 C CNN
-F 1 "GND" H 4950 3280 30  0001 C CNN
-F 2 "" H 4950 3350 60  0000 C CNN
-F 3 "" H 4950 3350 60  0000 C CNN
-	1    4950 3350
+P 4950 3150
+F 0 "#PWR1" H 4950 3150 30  0001 C CNN
+F 1 "GND" H 4950 3080 30  0001 C CNN
+F 2 "" H 4950 3150 60  0000 C CNN
+F 3 "" H 4950 3150 60  0000 C CNN
+	1    4950 3150
 	1    0    0    -1
 $EndComp
@@
 F 3 "" H 4500 3950 60  0000 C CNN
 	1    4500 3950
-	-1   0    0    -1
+	-1   0    0    1
 $EndComp
 $Comp
@@
 	4850 3250 5900 3250
 Wire Wire Line
-	4950 3250 4950 3350
-Wire Wire Line
 	4850 3050 6500 3050
 Wire Wire Line
@@
 Wire Wire Line
 	5750 4950 5750 4850
-Connection ~ 4950 3250
 Wire Notes Line
 	7050 2900 7050 3700
@@
 Wire Wire Line
 	6100 3850 6100 3550
+Wire Wire Line
+	4950 3050 4950 3150
+Connection ~ 4950 3050
+Text Notes 7100 3250 0    60   ~ 0
+Female\nbullets
+Text Notes 4250 3250 2    60   ~ 0
+Male\nbullets
 $EndSCHEMATC

Commit message: minor changes to sssw
Parts:
- D1: footprint (none) -> LEDs:LED-0805
- P1, P3: footprint (none) -> sssw:G3.5_Bullet_Edge_Short
- P2: footprint (none) -> Pin_Headers:Pin_Header_Angled_1x02
- Q1: footprint (none) -> Transistors_TO-220:TO-220_FET-GDS_Horizontal_LargePads
- R1, R2, R3: footprint (none) -> Resistors_SMD:Resistor_SMD0805_HandSoldering
Changed lines of the file:
@@
 LIBS:valves
 LIBS:sssw-cache
-EELAYER 24 0
+EELAYER 25 0
 EELAYER END
 $Descr A4 11693 8268
@@
 F 0 "Q1" H 6050 3500 60  0000 R CNN
 F 1 "SUP85" H 6050 3150 60  0000 R CNN
-F 2 "" H 6100 3350 60  0000 C CNN
+F 2 "Transistors_TO-220:TO-220_FET-GDS_Horizontal_LargePads" H 6100 3350 60  0001 C CNN
 F 3 "" H 6100 3350 60  0000 C CNN
 	1    6100 3350
@@
 F 0 "P1" V 4450 3150 40  0000 C CNN
 F 1 "INPUT" V 4550 3150 40  0000 C CNN
-F 2 "" H 4500 3150 60  0000 C CNN
+F 2 "sssw:G3.5_Bullet_Edge_Short" H 4500 3150 60  0001 C CNN
 F 3 "" H 4500 3150 60  0000 C CNN
 	1    4500 3150
@@
 F 0 "P3" V 6800 3150 40  0000 C CNN
 F 1 "OUTPUT" V 6900 3150 40  0000 C CNN
-F 2 "" H 6850 3150 60  0000 C CNN
+F 2 "sssw:G3.5_Bullet_Edge_Short" H 6850 3150 60  0001 C CNN
 F 3 "" H 6850 3150 60  0000 C CNN
 	1    6850 3150
@@
 F 0 "R1" V 5230 3850 40  0000 C CNN
 F 1 "10K" V 5157 3851 40  0000 C CNN
-F 2 "" V 5080 3850 30  0000 C CNN
+F 2 "Resistors_SMD:Resistor_SMD0805_HandSoldering" V 5080 3850 30  0001 C CNN
 F 3 "" H 5150 3850 30  0000 C CNN
 	1    5150 3850
@@
 F 0 "R2" V 5580 4150 40  0000 C CNN
 F 1 "1K" V 5507 4151 40  0000 C CNN
-F 2 "" V 5430 4150 30  0000 C CNN
+F 2 "Resistors_SMD:Resistor_SMD0805_HandSoldering" V 5430 4150 30  0001 C CNN
 F 3 "" H 5500 4150 30  0000 C CNN
 	1    5500 4150
@@
 F 0 "P2" V 4450 3950 40  0000 C CNN
 F 1 "ACTIVATE" V 4550 3950 40  0000 C CNN
-F 2 "" H 4500 3950 60  0000 C CNN
+F 2 "Pin_Headers:Pin_Header_Angled_1x02" H 4500 3950 60  0001 C CNN
 F 3 "" H 4500 3950 60  0000 C CNN
 	1    4500 3950
@@
 F 0 "D1" H 5750 4750 50  0000 C CNN
 F 1 "LED" H 5750 4550 50  0000 C CNN
-F 2 "" H 5750 4650 60  0000 C CNN
+F 2 "LEDs:LED-0805" H 5750 4650 60  0001 C CNN
 F 3 "" H 5750 4650 60  0000 C CNN
 	1    5750 4650
@@
 F 0 "R3" V 5830 4150 40  0000 C CNN
 F 1 "330" V 5757 4151 40  0000 C CNN
-F 2 "" V 5680 4150 30  0000 C CNN
+F 2 "Resistors_SMD:Resistor_SMD0805_HandSoldering" V 5680 4150 30  0001 C CNN
 F 3 "" H 5750 4150 30  0000 C CNN
 	1    5750 4150
